File: Routage.sch (KiCad schematic (older format))
At the start: 52 parts, among them J2 Conn_01x02, J3 Conn_01x03, Q1 2N2907, Q10 TIP32, Q11 BD138, Q12 TIP31, Q13 2N2222, Q2 2N2907, Q3 2N2907, Q4 2N2222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

Commit message: rajout_label
Parts:
- Dz1: symbol Device:BZX55C5V1 -> Routage-rescue:BZX55C5V1-Device
- U1: symbol Relay:Relay_1CT -> Routage-rescue:Relay_1CT-Relay
- U2: symbol Connector:Jack_Mono -> Routage-rescue:Jack_Mono-Connector
Connections:
- net Relay_Q13: now reaches D1.2 (A), Q13.3 (C), U1.b1
Changed lines of the file:
@@
 Connection ~ 2900 900
 $Comp
-L Relay:Relay_1CT U1
+L Routage-rescue:Relay_1CT-Relay U1
 U 1 1 5E9227D3
 P 9400 3250
@@
 	2400 1550 2400 1900
 $Comp
-L Device:BZX55C5V1 Dz1
+L Routage-rescue:BZX55C5V1-Device Dz1
 U 1 1 5E91152E
 P 2400 1400
@@
 	1600 3400 1900 3400
 $Comp
-L Connector:Jack_Mono U2
+L Routage-rescue:Jack_Mono-Connector U2
 U 1 1 5E8BA8E3
 P 850 3350
@@
 Text Label 2050 6650 0    50   ~ 0
 GND_Alim
+Text Label 9050 3750 0    50   ~ 0
+Relay_Q13
 $EndSCHEMATC
